File: hardware/kicad/usb_c_pd_power_board/01_usb_c_input.kicad_sch (KiCad schematic)
At the start: 1 part, among them J1 USB_C_Receptacle_USB2.0_16P

Commit message: complete MVP: Schematic & PCB Design
Parts:
- J1: footprint (none) -> Connector_USB:USB_C_Receptacle_GCT_USB4105-xx-A_16P_TopMnt_Horizontal
Changed lines of the file:
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@@
       (effects (font (size 1.27 1.27)))
     )
-    (property "Footprint" "" (at 146.05 90.17 0)
+    (property "Footprint" "Connector_USB:USB_C_Receptacle_GCT_USB4105-xx-A_16P_TopMnt_Horizontal" (at 146.05 90.17 0)
       (effects (font (size 1.27 1.27)) hide)
     )
