File: hardware/kicad/usb_c_pd_power_board/02_pd_controller.kicad_sch (KiCad schematic)
At the start: 8 parts, among them U1 STUSB4500QTR

Commit message: complete MVP: Schematic & PCB Design
Parts:
- C1, C2, C3, C4: footprint (none) -> Capacitor_SMD:C_0603_1608Metric
- R1, R2, R3: footprint (none) -> Resistor_SMD:R_0603_1608Metric
Changed lines of the file:
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@@
   (junction (at 127 116.84) (diameter 0) (color 0 0 0 0)
   )
+  (junction (at 142.24 121.92) (diameter 0) (color 0 0 0 0)
+  )
   (junction (at 125.73 111.76) (diameter 0) (color 0 0 0 0)
   )
@@
   )
   (junction (at 129.54 72.39) (diameter 0) (color 0 0 0 0)
+  )
+  (junction (at 142.24 76.2) (diameter 0) (color 0 0 0 0)
   )
   (wire (pts (xy 129.54 64.77) (xy 135.89 64.77))
@@
     )
   )
+  (symbol (lib_id "power:PWR_FLAG") (at 142.24 76.2 0) (unit 1)
+    (in_bom yes) (on_board yes) (dnp no) (fields_autoplaced)
+    (property "Reference" "#FLG03" (at 142.24 74.295 0)
+      (effects (font (size 1.27 1.27)) hide)
+    )
+    (property "Value" "PWR_FLAG" (at 142.24 71.12 0)
+      (effects (font (size 1.27 1.27)))
+    )
+    (property "Footprint" "" (at 142.24 76.2 0)
+      (effects (font (size 1.27 1.27)) hide)
+    )
+    (property "Datasheet" "~" (at 142.24 76.2 0)
+      (effects (font (size 1.27 1.27)) hide)
+    )
+    (pin "1")
+    (instances
+      (project "usb_c_pd_power_board"
+        (path "/f21e9372-3849-4e8f-9112-7a98c5af3538/22ba58ef-5eb5-4adf-ab03-440ed515c770"
+          (reference "#FLG03") (unit 1)
+        )
+      )
+    )
+  )
+  (symbol (lib_id "power:PWR_FLAG") (at 142.24 121.92 90) (unit 1)
+    (in_bom yes) (on_board yes) (dnp no) (fields_autoplaced)
+    (property "Reference" "#FLG04" (at 140.335 121.92 0)
+      (effects (font (size 1.27 1.27)) hide)
+    )
+    (property "Value" "PWR_FLAG" (at 138.43 121.92 90)
+      (effects (font (size 1.27 1.27)) (justify left))
+    )
+    (property "Footprint" "" (at 142.24 121.92 0)
+      (effects (font (size 1.27 1.27)) hide)
+    )
+    (property "Datasheet" "~" (at 142.24 121.92 0)
+      (effects (font (size 1.27 1.27)) hide)
+    )
+    (pin "1")
+    (instances
+      (project "usb_c_pd_power_board"
+        (path "/f21e9372-3849-4e8f-9112-7a98c5af3538/22ba58ef-5eb5-4adf-ab03-440ed515c770"
+          (reference "#FLG04") (unit 1)
+        )
+      )
+    )
+  )
   (symbol (lib_id "Device:R") (at 100.33 109.22 270) (unit 1)
     (in_bom yes) (on_board yes) (dnp no)
@@
       (effects (font (size 1.27 1.27)))
     )
-    (property "Footprint" "" (at 100.33 107.442 90)
+    (property "Footprint" "Resistor_SMD:R_0603_1608Metric" (at 100.33 107.442 90)
       (effects (font (size 1.27 1.27)) hide)
     )
@@
       (effects (font (size 1.27 1.27)) (justify left))
     )
-    (property "Footprint" "" (at 155.9052 72.39 0)
+    (property "Footprint" "Capacitor_SMD:C_0603_1608Metric" (at 155.9052 72.39 0)
       (effects (font (size 1.27 1.27)) hide)
     )
@@
       (effects (font (size 1.27 1.27)) (justify left))
     )
-    (property "Footprint" "" (at 122.682 76.2 90)
+    (property "Footprint" "Resistor_SMD:R_0603_1608Metric" (at 122.682 76.2 90)
       (effects (font (size 1.27 1.27)) hide)
     )
@@
       (effects (font (size 1.27 1.27)) (justify left))
     )
-    (property "Footprint" "" (at 130.5052 72.39 0)
+    (property "Footprint" "Capacitor_SMD:C_0603_1608Metric" (at 130.5052 72.39 0)
       (effects (font (size 1.27 1.27)) hide)
     )
@@
       (effects (font (size 1.27 1.27)) (justify right))
     )
-    (property "Footprint" "" (at 146.3548 64.77 0)
+    (property "Footprint" "Capacitor_SMD:C_0603_1608Metric" (at 146.3548 64.77 0)
       (effects (font (size 1.27 1.27)) hide)
     )
@@
       (effects (font (size 1.27 1.27)))
     )
-    (property "Footprint" "" (at 100.33 108.458 90)
+    (property "Footprint" "Resistor_SMD:R_0603_1608Metric" (at 100.33 108.458 90)
       (effects (font (size 1.27 1.27)) hide)
     )
@@
       (effects (font (size 1.27 1.27)) (justify left))
     )
-    (property "Footprint" "" (at 136.8552 72.39 0)
-      (effects (font (size 1.27 1.27)) hide)
-    )
+    (property "Footprint" "Capacitor_SMD:C_0603_1608Metric" (at 136.8552 72.39 0)
+      (effects (font (size 1.27 1.27)) hide)
+    )
