File: hardware/kicad/usb_c_pd_power_board/03_vbus_protection.kicad_sch (KiCad schematic)
At the start: 0 parts

Commit message: Add USB-C PD input power and 5V buck schematic
Parts:
- added C5: 10uF, symbol Device:C
- added C6, C8: 100nF, symbol Device:C
- added C7: 22uF, symbol Device:C
- added D1: SMBJ24A, symbol Device:D_Zener
- added F1: 3A Plyfuse, symbol Device:Fuse
- added Q1: DMP3098L, symbol Device:Q_PMOS_GDS
- added Q2, Q3: MMBT3904, symbol Device:Q_NPN_BEC
- added R4: 100k, symbol Device:R
- added R5: 10K, symbol Device:R
- added R6, R7: 10k, symbol Device:R
- added TP1, TP2, TP3, TP4: TestPoint, symbol Connector:TestPoint
Connections:
- new net: Q3.1 (B), R7.2
- new net: Q2.1 (B), R5.1
- new net GND: C5.2, C6.2, C7.2, C8.1, D1.1 (K), Q2.2 (E), Q3.2 (E)
- new net PD_DISCH: R7.1
- new net PD_DISCH_NODE: Q3.3 (C), R6.2
- new net PD_VBUS_EN: R5.2
- new net PD_VBUS_GATE: Q1.1 (G), Q2.3 (C), R4.2, TP4.1
- new net VBUS_FUSED: C5.1, C6.1, D1.2 (A), F1.2, Q1.3 (S), R4.1, TP2.1
- new net VBUS_PROTECTED: C7.1, C8.2, Q1.2 (D), R6.1, TP3.1
- new net VBUS_RAW: F1.1, TP1.1

Commit message: complete initial schematic and pass ERC
Changed lines of the file:
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@@
+    (effects (font (size 1.27 1.27)) (justify left bottom))
+  )
+  (label "PD_VBUS_GATE" (at 156.21 74.93 90) (fields_autoplaced)
     (effects (font (size 1.27 1.27)) (justify left bottom))
   )
@@
     (effects (font (size 1.27 1.27)) (justify left))
   )
-  (hierarchical_label "PD_VBUS_GATE" (shape input) (at 156.21 74.93 90) (fields_autoplaced)
-    (effects (font (size 1.27 1.27)) (justify left))
-  )

Commit message: complete MVP: Schematic & PCB Design
Parts:
- C5, C7: footprint (none) -> Capacitor_SMD:C_0805_2012Metric
- C6, C8: footprint (none) -> Capacitor_SMD:C_0603_1608Metric
- D1: footprint (none) -> Diode_SMD:D_SMB
- F1: footprint (none) -> Fuse:Fuse_1812_4532Metric
- Q1, Q2, Q3: footprint (none) -> Package_TO_SOT_SMD:SOT-23
- R4, R5, R6, R7: footprint (none) -> Resistor_SMD:R_0603_1608Metric
- TP1, TP2, TP3, TP4: footprint (none) -> TestPoint:TestPoint_Pad_D1.0mm
Changed lines of the file:
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@@
       (effects (font (size 1.27 1.27)))
     )
-    (property "Footprint" "" (at 105.41 85.598 90)
+    (property "Footprint" "Fuse:Fuse_1812_4532Metric" (at 105.41 85.598 90)
       (effects (font (size 1.27 1.27)) hide)
     )
@@
       (effects (font (size 1.27 1.27)) (justify left))
     )
-    (property "Footprint" "" (at 163.83 74.93 0)
+    (property "Footprint" "TestPoint:TestPoint_Pad_D1.0mm" (at 163.83 74.93 0)
       (effects (font (size 1.27 1.27)) hide)
     )
@@
       (effects (font (size 1.27 1.27)))
     )
-    (property "Footprint" "" (at 147.32 76.708 90)
+    (property "Footprint" "Resistor_SMD:R_0603_1608Metric" (at 147.32 76.708 90)
       (effects (font (size 1.27 1.27)) hide)
     )
@@
       (effects (font (size 1.27 1.27)))
     )
-    (property "Footprint" "" (at 177.8 90.4748 0)
+    (property "Footprint" "Capacitor_SMD:C_0805_2012Metric" (at 177.8 90.4748 0)
       (effects (font (size 1.27 1.27)) hide)
     )
@@
       (effects (font (size 1.27 1.27)))
     )
-    (property "Footprint" "" (at 161.29 106.68 0)
+    (property "Footprint" "Package_TO_SOT_SMD:SOT-23" (at 161.29 106.68 0)
       (effects (font (size 1.27 1.27)) hide)
     )
@@
       (effects (font (size 1.27 1.27)))
     )
-    (property "Footprint" "" (at 186.69 72.39 0)
+    (property "Footprint" "Package_TO_SOT_SMD:SOT-23" (at 186.69 72.39 0)
       (effects (font (size 1.27 1.27)) hide)
     )
@@
       (effects (font (size 1.27 1.27)) (justify right))
     )
-    (property "Footprint" "" (at 134.62 91.44 0)
+    (property "Footprint" "Diode_SMD:D_SMB" (at 134.62 91.44 0)
       (effects (font (size 1.27 1.27)) hide)
     )
@@
       (effects (font (size 1.27 1.27)) (justify right))
     )
-    (property "Footprint" "" (at 92.71 83.82 0)
+    (property "Footprint" "TestPoint:TestPoint_Pad_D1.0mm" (at 92.71 83.82 0)
       (effects (font (size 1.27 1.27)) hide)
     )
@@
       (effects (font (size 1.27 1.27)) (justify right))
     )
-    (property "Footprint" "" (at 157.48 83.82 0)
+    (property "Footprint" "TestPoint:TestPoint_Pad_D1.0mm" (at 157.48 83.82 0)
       (effects (font (size 1.27 1.27)) hide)
     )
@@
       (effects (font (size 1.27 1.27)) (justify left))
     )
-    (property "Footprint" "" (at 187.452 90.17 90)
+    (property "Footprint" "Resistor_SMD:R_0603_1608Metric" (at 187.452 90.17 90)
       (effects (font (size 1.27 1.27)) hide)
     )
@@
       (effects (font (size 1.27 1.27)) (justify left))
     )
-    (property "Footprint" "" (at 168.402 97.79 90)
+    (property "Footprint" "Resistor_SMD:R_0603_1608Metric" (at 168.402 97.79 90)
       (effects (font (size 1.27 1.27)) hide)
     )
@@
       (effects (font (size 1.27 1.27)))
     )
-    (property "Footprint" "" (at 154.94 98.298 90)
+    (property "Footprint" "Resistor_SMD:R_0603_1608Metric" (at 154.94 98.298 90)
       (effects (font (size 1.27 1.27)) hide)
     )
@@
       (effects (font (size 1.27 1.27)) (justify left))
     )
-    (property "Footprint" "" (at 124.1552 95.25 0)
+    (property "Footprint" "Capacitor_SMD:C_0805_2012Metric" (at 124.1552 95.25 0)
       (effects (font (size 1.27 1.27)) hide)
     )
@@
       (effects (font (size 1.27 1.27)))
     )
-    (property "Footprint" "" (at 170.18 84.7852 0)
+    (property "Footprint" "Capacitor_SMD:C_0603_1608Metric" (at 170.18 84.7852 0)
       (effects (font (size 1.27 1.27)) hide)
     )
@@
       (effects (font (size 1.27 1.27)) (justify left))
     )
-    (property "Footprint" "" (at 112.7252 95.25 0)
+    (property "Footprint" "Capacitor_SMD:C_0603_1608Metric" (at 112.7252 95.25 0)
       (effects (font (size 1.27 1.27)) hide)
     )
@@
       (effects (font (size 1.27 1.27)))
     )
-    (property "Footprint" "" (at 158.75 86.36 0)
+    (property "Footprint" "Package_TO_SOT_SMD:SOT-23" (at 158.75 86.36 0)
       (effects (font (size 1.27 1.27)) hide)
     )
@@
       (effects (font (size 1.27 1.27)) (justify left))
     )
-    (property "Footprint" "" (at 116.84 83.82 0)
-      (effects (font (size 1.27 1.27)) hide)
-    )
+    (property "Footprint" "TestPoint:TestPoint_Pad_D1.0mm" (at 116.84 83.82 0)
+      (effects (font (size 1.27 1.27)) hide)
+    )
