File: hardware/kicad/usb_c_pd_power_board/06_output_connectors.kicad_sch (KiCad schematic)
At the start: 0 parts

Commit message: complete initial schematic and pass ERC
Parts:
- added J2: 5V_OUT, symbol Connector_Generic:Conn_01x02
- added J3: 3V3_OUT, symbol Connector_Generic:Conn_01x02
- added J4: VBUS_PROTECTED_OUT, symbol Connector_Generic:Conn_01x02
- added J5: Conn_01x04, symbol Connector_Generic:Conn_01x04
Connections:
- new net +3V3: J3.1 (Pin_1), J5.3 (Pin_3)
- new net +5V: J2.1 (Pin_1), J5.2 (Pin_2)
- new net GND: J2.2 (Pin_2), J3.2 (Pin_2), J4.2 (Pin_2), J5.4 (Pin_4)
- new net VBUS_PROTECTED: J4.1 (Pin_1), J5.1 (Pin_1)
Changed lines of the file:
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@@
 (kicad_sch (version 20230121) (generator eeschema)
   (paper "A4")
+  (wire (pts (xy 115.57 78.74) (xy 115.57 81.28))
+    (stroke (width 0) (type default))
+  )
+  (wire (pts (xy 136.525 78.74) (xy 136.525 81.28))
+    (stroke (width 0) (type default))
+  )
+  (wire (pts (xy 176.53 78.74) (xy 176.53 81.915))
+    (stroke (width 0) (type default))
+  )
+  (wire (pts (xy 96.52 78.74) (xy 96.52 81.28))
+    (stroke (width 0) (type default))
+  )
+  (wire (pts (xy 93.98 78.74) (xy 93.98 81.28))
+    (stroke (width 0) (type default))
+  )
+  (wire (pts (xy 168.91 78.74) (xy 168.91 81.915))
+    (stroke (width 0) (type default))
+  )
+  (wire (pts (xy 173.99 78.74) (xy 173.99 81.915))
+    (stroke (width 0) (type default))
+  )
+  (wire (pts (xy 133.985 78.74) (xy 133.985 81.28))
+    (stroke (width 0) (type default))
+  )
+  (wire (pts (xy 113.03 78.74) (xy 113.03 81.28))
+    (stroke (width 0) (type default))
+  )
+  (wire (pts (xy 171.45 78.74) (xy 171.45 81.915))
+    (stroke (width 0) (type default))
+  )
+  (hierarchical_label "+3V3" (shape input) (at 113.03 81.28 270) (fields_autoplaced)
+    (effects (font (size 1.27 1.27)) (justify right))
+  )
+  (hierarchical_label "+3V3" (shape input) (at 173.99 81.915 270) (fields_autoplaced)
+    (effects (font (size 1.27 1.27)) (justify right))
+  )
+  (hierarchical_label "VBUS_PROTECTED" (shape input) (at 133.985 81.28 270) (fields_autoplaced)
+    (effects (font (size 1.27 1.27)) (justify right))
+  )
+  (hierarchical_label "+5V" (shape input) (at 93.98 81.28 270) (fields_autoplaced)
+    (effects (font (size 1.27 1.27)) (justify right))
+  )
+  (hierarchical_label "VBUS_PROTECTED" (shape input) (at 168.91 81.915 270) (fields_autoplaced)
+    (effects (font (size 1.27 1.27)) (justify right))
+  )
+  (hierarchical_label "GND" (shape input) (at 115.57 81.28 270) (fields_autoplaced)
+    (effects (font (size 1.27 1.27)) (justify right))
+  )
+  (hierarchical_label "+5V" (shape input) (at 171.45 81.915 270) (fields_autoplaced)
+    (effects (font (size 1.27 1.27)) (justify right))
+  )
+  (hierarchical_label "GND" (shape input) (at 136.525 81.28 270) (fields_autoplaced)
+    (effects (font (size 1.27 1.27)) (justify right))
+  )
+  (hierarchical_label "GND" (shape input) (at 176.53 81.915 270) (fields_autoplaced)
+    (effects (font (size 1.27 1.27)) (justify right))
+  )
+  (hierarchical_label "GND" (shape input) (at 96.52 81.28 270) (fields_autoplaced)
+    (effects (font (size 1.27 1.27)) (justify right))
+  )
+  (symbol (lib_id "Connector_Generic:Conn_01x02") (at 113.03 73.66 90) (unit 1)
+    (in_bom yes) (on_board yes) (dnp no) (fields_autoplaced)
+    (property "Reference" "J3" (at 118.11 72.39 90)
+      (effects (font (size 1.27 1.27)) (justify right))
+    )
+    (property "Value" "3V3_OUT" (at 118.11 74.93 90)
+      (effects (font (size 1.27 1.27)) (justify right))
+    )
+    (property "Footprint" "" (at 113.03 73.66 0)
+      (effects (font (size 1.27 1.27)) hide)
+    )
+    (property "Datasheet" "~" (at 113.03 73.66 0)
+      (effects (font (size 1.27 1.27)) hide)
+    )
+    (pin "2")
+    (pin "1")
+    (instances
+      (project "usb_c_pd_power_board"
+        (path "/f21e9372-3849-4e8f-9112-7a98c5af3538/2a9ff4ab-2886-479e-950c-fea96f57bac3"
+          (reference "J3") (unit 1)
+        )
+      )
+    )
+  )
+  (symbol (lib_id "Connector_Generic:Conn_01x02") (at 93.98 73.66 90) (unit 1)
+    (in_bom yes) (on_board yes) (dnp no) (fields_autoplaced)
+    (property "Reference" "J2" (at 99.06 72.39 90)
+      (effects (font (size 1.27 1.27)) (justify right))
+    )
+    (property "Value" "5V_OUT" (at 99.06 74.93 90)
+      (effects (font (size 1.27 1.27)) (justify right))
+    )
+    (property "Footprint" "" (at 93.98 73.66 0)
+      (effects (font (size 1.27 1.27)) hide)
+    )
+    (property "Datasheet" "~" (at 93.98 73.66 0)
+      (effects (font (size 1.27 1.27)) hide)
+    )
+    (pin "1")
+    (pin "2")
+    (instances
+      (project "usb_c_pd_power_board"
+        (path "/f21e9372-3849-4e8f-9112-7a98c5af3538/2a9ff4ab-2886-479e-950c-fea96f57bac3"
+          (reference "J2") (unit 1)
+        )
+      )
+    )
+  )
+  (symbol (lib_id "Connector_Generic:Conn_01x04") (at 171.45 73.66 90) (unit 1)
+    (in_bom yes) (on_board yes) (dnp no) (fields_autoplaced)
+    (property "Reference" "J5" (at 172.72 67.31 90)
+      (effects (font (size 1.27 1.27)))
+    )
+    (property "Value" "Conn_01x04" (at 172.72 69.85 90)
+      (effects (font (size 1.27 1.27)))
+    )
+    (property "Footprint" "" (at 171.45 73.66 0)
+      (effects (font (size 1.27 1.27)) hide)
+    )
+    (property "Datasheet" "~" (at 171.45 73.66 0)
+      (effects (font (size 1.27 1.27)) hide)
+    )
+    (pin "4")
+    (pin "2")
+    (pin "3")
+    (pin "1")
+    (instances
+      (project "usb_c_pd_power_board"
+        (path "/f21e9372-3849-4e8f-9112-7a98c5af3538/2a9ff4ab-2886-479e-950c-fea96f57bac3"
+          (reference "J5") (unit 1)
+        )
+      )
+    )
+  )
+  (symbol (lib_id "Connector_Generic:Conn_01x02") (at 133.985 73.66 90) (unit 1)
+    (in_bom yes) (on_board yes) (dnp no) (fields_autoplaced)
+    (property "Reference" "J4" (at 139.7 72.39 90)
+      (effects (font (size 1.27 1.27)) (justify right))
+    )
+    (property "Value" "VBUS_PROTECTED_OUT" (at 139.7 74.93 90)
+      (effects (font (size 1.27 1.27)) (justify right))
+    )
+    (property "Footprint" "" (at 133.985 73.66 0)
+      (effects (font (size 1.27 1.27)) hide)
+    )
+    (property "Datasheet" "~" (at 133.985 73.66 0)
+      (effects (font (size 1.27 1.27)) hide)
+    )
+    (pin "2")
+    (pin "1")
+    (instances
+      (project "usb_c_pd_power_board"
+        (path "/f21e9372-3849-4e8f-9112-7a98c5af3538/2a9ff4ab-2886-479e-950c-fea96f57bac3"
+          (reference "J4") (unit 1)
+        )
+      )
+    )
+  )
 )

Commit message: complete MVP: Schematic & PCB Design
Parts:
- J2, J3, J4: footprint (none) -> Connector_PinHeader_2.54mm:PinHeader_1x02_P2.54mm_Vertical
- J5: footprint (none) -> Connector_PinHeader_2.54mm:PinHeader_1x04_P2.54mm_Vertical
Changed lines of the file:
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@@
       (effects (font (size 1.27 1.27)) (justify right))
     )
-    (property "Footprint" "" (at 113.03 73.66 0)
+    (property "Footprint" "Connector_PinHeader_2.54mm:PinHeader_1x02_P2.54mm_Vertical" (at 113.03 73.66 0)
       (effects (font (size 1.27 1.27)) hide)
     )
@@
       (effects (font (size 1.27 1.27)) (justify right))
     )
-    (property "Footprint" "" (at 93.98 73.66 0)
+    (property "Footprint" "Connector_PinHeader_2.54mm:PinHeader_1x02_P2.54mm_Vertical" (at 93.98 73.66 0)
       (effects (font (size 1.27 1.27)) hide)
     )
@@
       (effects (font (size 1.27 1.27)))
     )
-    (property "Footprint" "" (at 171.45 73.66 0)
+    (property "Footprint" "Connector_PinHeader_2.54mm:PinHeader_1x04_P2.54mm_Vertical" (at 171.45 73.66 0)
       (effects (font (size 1.27 1.27)) hide)
     )
@@
       (effects (font (size 1.27 1.27)) (justify right))
     )
-    (property "Footprint" "" (at 133.985 73.66 0)
+    (property "Footprint" "Connector_PinHeader_2.54mm:PinHeader_1x02_P2.54mm_Vertical" (at 133.985 73.66 0)
       (effects (font (size 1.27 1.27)) hide)
     )
