File: hardware/kicad/usb_c_pd_power_board/07_status_leds.kicad_sch (KiCad schematic)
At the start: 0 parts

Commit message: complete initial schematic and pass ERC
Parts:
- added D2: 5V_OK, symbol Device:LED
- added D3: 3V3_OK, symbol Device:LED
- added D4: PD_ATTACH, symbol Device:LED
- added R10: 2.2k, symbol Device:R
- added R11, R12: 1k, symbol Device:R
Connections:
- new net: D2.2 (A), R10.2
- new net: D4.2 (A), R12.2
- new net: D3.2 (A), R11.2
- new net +3V3: R11.1
- new net +5V: R10.1
- new net GND: D2.1 (K), D3.1 (K), D4.1 (K)
- new net PD_ATTACH: R12.1
Changed lines of the file:
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@@
 (kicad_sch (version 20230121) (generator eeschema)
   (paper "A4")
+  (wire (pts (xy 143.51 98.425) (xy 143.51 103.505))
+    (stroke (width 0) (type default))
+  )
+  (wire (pts (xy 180.975 98.425) (xy 180.975 102.87))
+    (stroke (width 0) (type default))
+  )
+  (wire (pts (xy 143.51 87.63) (xy 143.51 90.805))
+    (stroke (width 0) (type default))
+  )
+  (wire (pts (xy 180.975 74.93) (xy 180.975 80.01))
+    (stroke (width 0) (type default))
+  )
+  (wire (pts (xy 160.655 87.63) (xy 160.655 90.805))
+    (stroke (width 0) (type default))
+  )
+  (wire (pts (xy 160.655 75.565) (xy 160.655 80.01))
+    (stroke (width 0) (type default))
+  )
+  (wire (pts (xy 143.51 76.835) (xy 143.51 80.01))
+    (stroke (width 0) (type default))
+  )
+  (wire (pts (xy 180.975 87.63) (xy 180.975 90.805))
+    (stroke (width 0) (type default))
+  )
+  (wire (pts (xy 160.655 98.425) (xy 160.655 103.505))
+    (stroke (width 0) (type default))
+  )
+  (hierarchical_label "GND" (shape input) (at 160.655 103.505 270) (fields_autoplaced)
+    (effects (font (size 1.27 1.27)) (justify right))
+  )
+  (hierarchical_label "GND" (shape input) (at 143.51 103.505 270) (fields_autoplaced)
+    (effects (font (size 1.27 1.27)) (justify right))
+  )
+  (hierarchical_label "GND" (shape input) (at 180.975 102.87 270) (fields_autoplaced)
+    (effects (font (size 1.27 1.27)) (justify right))
+  )
+  (hierarchical_label "+5V" (shape input) (at 143.51 76.835 90) (fields_autoplaced)
+    (effects (font (size 1.27 1.27)) (justify left))
+  )
+  (hierarchical_label "PD_ATTACH" (shape input) (at 180.975 74.93 90) (fields_autoplaced)
+    (effects (font (size 1.27 1.27)) (justify left))
+  )
+  (hierarchical_label "+3V3" (shape input) (at 160.655 75.565 90) (fields_autoplaced)
+    (effects (font (size 1.27 1.27)) (justify left))
+  )
+  (symbol (lib_id "Device:LED") (at 143.51 94.615 90) (unit 1)
+    (in_bom yes) (on_board yes) (dnp no) (fields_autoplaced)
+    (property "Reference" "D2" (at 147.32 94.9325 90)
+      (effects (font (size 1.27 1.27)) (justify right))
+    )
+    (property "Value" "5V_OK" (at 147.32 97.4725 90)
+      (effects (font (size 1.27 1.27)) (justify right))
+    )
+    (property "Footprint" "" (at 143.51 94.615 0)
+      (effects (font (size 1.27 1.27)) hide)
+    )
+    (property "Datasheet" "~" (at 143.51 94.615 0)
+      (effects (font (size 1.27 1.27)) hide)
+    )
+    (pin "2")
+    (pin "1")
+    (instances
+      (project "usb_c_pd_power_board"
+        (path "/f21e9372-3849-4e8f-9112-7a98c5af3538/4e6ca347-cc69-4a2a-ba48-e5b8a0f48b51"
+          (reference "D2") (unit 1)
+        )
+      )
+    )
+  )
+  (symbol (lib_id "Device:LED") (at 180.975 94.615 90) (unit 1)
+    (in_bom yes) (on_board yes) (dnp no) (fields_autoplaced)
+    (property "Reference" "D4" (at 184.15 94.9325 90)
+      (effects (font (size 1.27 1.27)) (justify right))
+    )
+    (property "Value" "PD_ATTACH" (at 184.15 97.4725 90)
+      (effects (font (size 1.27 1.27)) (justify right))
+    )
+    (property "Footprint" "" (at 180.975 94.615 0)
+      (effects (font (size 1.27 1.27)) hide)
+    )
+    (property "Datasheet" "~" (at 180.975 94.615 0)
+      (effects (font (size 1.27 1.27)) hide)
+    )
+    (pin "2")
+    (pin "1")
+    (instances
+      (project "usb_c_pd_power_board"
+        (path "/f21e9372-3849-4e8f-9112-7a98c5af3538/4e6ca347-cc69-4a2a-ba48-e5b8a0f48b51"
+          (reference "D4") (unit 1)
+        )
+      )
+    )
+  )
+  (symbol (lib_id "Device:R") (at 160.655 83.82 0) (unit 1)
+    (in_bom yes) (on_board yes) (dnp no) (fields_autoplaced)
+    (property "Reference" "R11" (at 162.56 82.55 0)
+      (effects (font (size 1.27 1.27)) (justify left))
+    )
+    (property "Value" "1k" (at 162.56 85.09 0)
+      (effects (font (size 1.27 1.27)) (justify left))
+    )
+    (property "Footprint" "" (at 158.877 83.82 90)
+      (effects (font (size 1.27 1.27)) hide)
+    )
+    (property "Datasheet" "~" (at 160.655 83.82 0)
+      (effects (font (size 1.27 1.27)) hide)
+    )
+    (pin "2")
+    (pin "1")
+    (instances
+      (project "usb_c_pd_power_board"
+        (path "/f21e9372-3849-4e8f-9112-7a98c5af3538/4e6ca347-cc69-4a2a-ba48-e5b8a0f48b51"
+          (reference "R11") (unit 1)
+        )
+      )
+    )
+  )
+  (symbol (lib_id "Device:R") (at 143.51 83.82 0) (unit 1)
+    (in_bom yes) (on_board yes) (dnp no) (fields_autoplaced)
+    (property "Reference" "R10" (at 145.415 82.55 0)
+      (effects (font (size 1.27 1.27)) (justify left))
+    )
+    (property "Value" "2.2k" (at 145.415 85.09 0)
+      (effects (font (size 1.27 1.27)) (justify left))
+    )
+    (property "Footprint" "" (at 141.732 83.82 90)
+      (effects (font (size 1.27 1.27)) hide)
+    )
+    (property "Datasheet" "~" (at 143.51 83.82 0)
+      (effects (font (size 1.27 1.27)) hide)
+    )
+    (pin "2")
+    (pin "1")
+    (instances
+      (project "usb_c_pd_power_board"
+        (path "/f21e9372-3849-4e8f-9112-7a98c5af3538/4e6ca347-cc69-4a2a-ba48-e5b8a0f48b51"
+          (reference "R10") (unit 1)
+        )
+      )
+    )
+  )
+  (symbol (lib_id "Device:LED") (at 160.655 94.615 90) (unit 1)
+    (in_bom yes) (on_board yes) (dnp no) (fields_autoplaced)
+    (property "Reference" "D3" (at 163.83 94.9325 90)
+      (effects (font (size 1.27 1.27)) (justify right))
+    )
+    (property "Value" "3V3_OK" (at 163.83 97.4725 90)
+      (effects (font (size 1.27 1.27)) (justify right))
+    )
+    (property "Footprint" "" (at 160.655 94.615 0)
+      (effects (font (size 1.27 1.27)) hide)
+    )
+    (property "Datasheet" "~" (at 160.655 94.615 0)
+      (effects (font (size 1.27 1.27)) hide)
+    )
+    (pin "2")
+    (pin "1")
+    (instances
+      (project "usb_c_pd_power_board"
+        (path "/f21e9372-3849-4e8f-9112-7a98c5af3538/4e6ca347-cc69-4a2a-ba48-e5b8a0f48b51"
+          (reference "D3") (unit 1)
+        )
+      )
+    )
+  )
+  (symbol (lib_id "Device:R") (at 180.975 83.82 0) (unit 1)
+    (in_bom yes) (on_board yes) (dnp no) (fields_autoplaced)
+    (property "Reference" "R12" (at 182.88 82.55 0)
+      (effects (font (size 1.27 1.27)) (justify left))
+    )
+    (property "Value" "1k" (at 182.88 85.09 0)
+      (effects (font (size 1.27 1.27)) (justify left))
+    )
+    (property "Footprint" "" (at 179.197 83.82 90)
+      (effects (font (size 1.27 1.27)) hide)
+    )
+    (property "Datasheet" "~" (at 180.975 83.82 0)
+      (effects (font (size 1.27 1.27)) hide)
+    )
+    (pin "2")
+    (pin "1")
+    (instances
+      (project "usb_c_pd_power_board"
+        (path "/f21e9372-3849-4e8f-9112-7a98c5af3538/4e6ca347-cc69-4a2a-ba48-e5b8a0f48b51"
+          (reference "R12") (unit 1)
+        )
+      )
+    )
+  )
 )

Commit message: complete MVP: Schematic & PCB Design
Parts:
- D2, D3, D4: footprint (none) -> LED_SMD:LED_0603_1608Metric
- R10, R11, R12: footprint (none) -> Resistor_SMD:R_0603_1608Metric
Changed lines of the file:
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@@
       (effects (font (size 1.27 1.27)) (justify right))
     )
-    (property "Footprint" "" (at 143.51 94.615 0)
+    (property "Footprint" "LED_SMD:LED_0603_1608Metric" (at 143.51 94.615 0)
       (effects (font (size 1.27 1.27)) hide)
     )
@@
       (effects (font (size 1.27 1.27)) (justify right))
     )
-    (property "Footprint" "" (at 180.975 94.615 0)
+    (property "Footprint" "LED_SMD:LED_0603_1608Metric" (at 180.975 94.615 0)
       (effects (font (size 1.27 1.27)) hide)
     )
@@
       (effects (font (size 1.27 1.27)) (justify left))
     )
-    (property "Footprint" "" (at 158.877 83.82 90)
+    (property "Footprint" "Resistor_SMD:R_0603_1608Metric" (at 158.877 83.82 90)
       (effects (font (size 1.27 1.27)) hide)
     )
@@
       (effects (font (size 1.27 1.27)) (justify left))
     )
-    (property "Footprint" "" (at 141.732 83.82 90)
+    (property "Footprint" "Resistor_SMD:R_0603_1608Metric" (at 141.732 83.82 90)
       (effects (font (size 1.27 1.27)) hide)
     )
@@
       (effects (font (size 1.27 1.27)) (justify right))
     )
-    (property "Footprint" "" (at 160.655 94.615 0)
+    (property "Footprint" "LED_SMD:LED_0603_1608Metric" (at 160.655 94.615 0)
       (effects (font (size 1.27 1.27)) hide)
     )
@@
       (effects (font (size 1.27 1.27)) (justify left))
     )
-    (property "Footprint" "" (at 179.197 83.82 90)
+    (property "Footprint" "Resistor_SMD:R_0603_1608Metric" (at 179.197 83.82 90)
       (effects (font (size 1.27 1.27)) hide)
     )
