File: hardware/kicad/usb_c_pd_power_board/08_test_points.kicad_sch (KiCad schematic)
At the start: 0 parts

Commit message: complete initial schematic and pass ERC
Parts:
- added TP10: VBUS_RAW, symbol Connector:TestPoint
- added TP11: VBUS_FUSED, symbol Connector:TestPoint
- added TP12: VBUS_PROTECTED, symbol Connector:TestPoint
- added TP13: +5V, symbol Connector:TestPoint
- added TP14: +3V3, symbol Connector:TestPoint
- added TP15: GND, symbol Connector:TestPoint
- added TP16: PD_VBUS_EN, symbol Connector:TestPoint
- added TP17: PD_DISCH, symbol Connector:TestPoint
- added TP18: PD_ATTACH, symbol Connector:TestPoint
- added TP19: PD_ALERT, symbol Connector:TestPoint
- added TP20: I2C_SCL, symbol Connector:TestPoint
- added TP21: I2C_SDA, symbol Connector:TestPoint
Connections:
- new net +3V3: TP14.1
- new net +5V: TP13.1
- new net GND: TP15.1
- new net I2C_SCL: TP20.1
- new net I2C_SDA: TP21.1
- new net PD_ALERT: TP19.1
- new net PD_ATTACH: TP18.1
- new net PD_DISCH: TP17.1
- new net PD_VBUS_EN: TP16.1
- new net VBUS_FUSED: TP11.1
- new net VBUS_PROTECTED: TP12.1
- new net VBUS_RAW: TP10.1

Commit message: complete MVP: Schematic & PCB Design
Parts:
- TP10, TP11, TP12, TP13, TP14, TP15, TP16, TP17, TP18, TP19, TP20, TP21: footprint (none) -> TestPoint:TestPoint_Pad_D1.0mm
Changed lines of the file:
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@@
       (effects (font (size 1.27 1.27)) (justify left))
     )
-    (property "Footprint" "" (at 117.475 105.41 0)
+    (property "Footprint" "TestPoint:TestPoint_Pad_D1.0mm" (at 117.475 105.41 0)
       (effects (font (size 1.27 1.27)) hide)
     )
@@
       (effects (font (size 1.27 1.27)) (justify left))
     )
-    (property "Footprint" "" (at 116.84 90.17 0)
+    (property "Footprint" "TestPoint:TestPoint_Pad_D1.0mm" (at 116.84 90.17 0)
       (effects (font (size 1.27 1.27)) hide)
     )
@@
       (effects (font (size 1.27 1.27)) (justify left))
     )
-    (property "Footprint" "" (at 117.475 97.79 0)
+    (property "Footprint" "TestPoint:TestPoint_Pad_D1.0mm" (at 117.475 97.79 0)
       (effects (font (size 1.27 1.27)) hide)
     )
@@
       (effects (font (size 1.27 1.27)) (justify left))
     )
-    (property "Footprint" "" (at 154.94 88.9 0)
+    (property "Footprint" "TestPoint:TestPoint_Pad_D1.0mm" (at 154.94 88.9 0)
       (effects (font (size 1.27 1.27)) hide)
     )
@@
       (effects (font (size 1.27 1.27)) (justify left))
     )
-    (property "Footprint" "" (at 154.305 81.28 0)
+    (property "Footprint" "TestPoint:TestPoint_Pad_D1.0mm" (at 154.305 81.28 0)
       (effects (font (size 1.27 1.27)) hide)
     )
@@
       (effects (font (size 1.27 1.27)) (justify left))
     )
-    (property "Footprint" "" (at 155.575 111.125 0)
+    (property "Footprint" "TestPoint:TestPoint_Pad_D1.0mm" (at 155.575 111.125 0)
       (effects (font (size 1.27 1.27)) hide)
     )
@@
       (effects (font (size 1.27 1.27)) (justify left))
     )
-    (property "Footprint" "" (at 154.94 103.505 0)
+    (property "Footprint" "TestPoint:TestPoint_Pad_D1.0mm" (at 154.94 103.505 0)
       (effects (font (size 1.27 1.27)) hide)
     )
@@
       (effects (font (size 1.27 1.27)) (justify left))
     )
-    (property "Footprint" "" (at 116.84 81.915 0)
+    (property "Footprint" "TestPoint:TestPoint_Pad_D1.0mm" (at 116.84 81.915 0)
       (effects (font (size 1.27 1.27)) hide)
     )
@@
       (effects (font (size 1.27 1.27)) (justify left))
     )
-    (property "Footprint" "" (at 154.94 96.52 0)
+    (property "Footprint" "TestPoint:TestPoint_Pad_D1.0mm" (at 154.94 96.52 0)
       (effects (font (size 1.27 1.27)) hide)
     )
@@
       (effects (font (size 1.27 1.27)) (justify left))
     )
-    (property "Footprint" "" (at 117.475 120.65 0)
+    (property "Footprint" "TestPoint:TestPoint_Pad_D1.0mm" (at 117.475 120.65 0)
       (effects (font (size 1.27 1.27)) hide)
     )
@@
       (effects (font (size 1.27 1.27)) (justify left))
     )
-    (property "Footprint" "" (at 155.575 119.38 0)
+    (property "Footprint" "TestPoint:TestPoint_Pad_D1.0mm" (at 155.575 119.38 0)
       (effects (font (size 1.27 1.27)) hide)
     )
@@
       (effects (font (size 1.27 1.27)) (justify left))
     )
-    (property "Footprint" "" (at 117.475 113.03 0)
-      (effects (font (size 1.27 1.27)) hide)
-    )
+    (property "Footprint" "TestPoint:TestPoint_Pad_D1.0mm" (at 117.475 113.03 0)
+      (effects (font (size 1.27 1.27)) hide)
+    )
